Commit message: robot petmodel implemented

File: urdf/robot.xacro (robot description, xacro)
@@ -1,19 +1,19 @@
 <?xml version="1.0"?>
 <robot xmlns:xacro="http://www.ros.org/wiki/xacro" name="robot_xacro">
-<xacro:include filename="$(find exp_assignment2)/urdf/robot.gazebo"/>
-	<xacro:property name="length_wheel" value="0.04" />
-	<xacro:property name="radius_wheel" value="0.1" />
-	<xacro:macro name="default_inertial" params="mass">
-               <inertial>
-                       <mass value="${mass}" />
-                       <origin rpy="0 1.5707 1.5707" xyz="0 0 0"/>
-                       <inertia ixx="0.000526666666667" ixy="0" ixz="0" iyy="0.000526666666667" iyz="0" izz="0.001"/>
-               </inertial>
-	</xacro:macro>
-    <xacro:macro name="wheel_geometry">
-		<geometry>
-       			<cylinder length="${length_wheel}" radius="${radius_wheel}"/>
-     	</geometry>
-	</xacro:macro>
+  <xacro:include filename="$(find exp_assignment2)/urdf/robot.gazebo"/>
+  <xacro:property name="length_wheel" value="0.04" />
+  <xacro:property name="radius_wheel" value="0.1" />
+  <xacro:macro name="default_inertial" params="mass">
+    <inertial>
+      <mass value="${mass}" />
+      <origin rpy="0 1.5707 1.5707" xyz="0 0 0"/>
+      <inertia ixx="0.000526666666667" ixy="0" ixz="0" iyy="0.000526666666667" iyz="0" izz="0.001"/>
+    </inertial>
+  </xacro:macro>
+  <xacro:macro name="wheel_geometry">
+    <geometry>
+      <cylinder length="${length_wheel}" radius="${radius_wheel}"/>
+    </geometry>
+  </xacro:macro>
   <material name="black">
     <color rgba="0.0 0.0 0.0 1.0"/>
@@ -40,5 +40,5 @@
     <color rgba="1.0 1.0 1.0 1.0"/>
   </material>
-	  <link name="link_chassis">
+  <link name="link_chassis">
     <!-- pose and inertial -->
     <pose>0 0 0.1 0 0 0</pose>
@@ -75,5 +75,5 @@
     </visual>
   </link>
-   <link name="link_right_wheel">
+  <link name="link_right_wheel">
     <xacro:default_inertial mass="0.2"/>
     <collision name="link_right_wheel_collision">
@@ -87,5 +87,5 @@
     </visual>
   </link>
-   <link name="link_left_wheel">
+  <link name="link_left_wheel">
     <xacro:default_inertial mass="0.2"/>
     <collision name="link_left_wheel_collision">
@@ -115,31 +115,57 @@
     <joint_properties damping="1.0" friction="1.0"/>
   </joint>
+  <link name="neck_link">
+    <collision>
+      <origin xyz="0 0 0.05" rpy="0 0 0"/>
+      <geometry>
+        <cylinder radius="0.04" length="0.1"/>
+      </geometry>
+    </collision>
+    <visual>
+      <origin xyz="0 0 0.05" rpy="0 0 0"/>
+      <geometry>
+        <cylinder radius="0.04" length="0.1"/>
+      </geometry>
+      <material name="orange"/>
+    </visual>
+    <inertial>
+      <mass value="1e-5" />
+      <origin xyz="0 0 0" rpy="0 0 0"/>
+      <inertia ixx="1e-6" ixy="0" ixz="0" iyy="1e-6" iyz="0" izz="1e-6" />
+    </inertial>
+  </link>
+  <joint name="neck_joint" type="fixed">
+    <axis xyz="0 1 0" />
+    <origin xyz="0.2 0 0.035" rpy="0 0 0"/>
+    <parent link="link_chassis"/>
+    <child link="neck_link"/>
+  </joint>
   <link name="camera_link">
-	    <collision>
-	      <origin xyz="0 0 0.025" rpy="0 0 0"/>
-	      <geometry>
-		<box size="0.05 0.05 0.05"/>
-	      </geometry>
-	    </collision>
-	    <visual>
-	      <origin xyz="0 0 0.025" rpy="0 0 0"/>
-	      <geometry>
-		<box size="0.05 0.05 0.05"/>
-	      </geometry>
-	      <material name="red">
-		<color rgba="1 0 0 1"/>
-	      </material>
-	    </visual>
-	    <inertial>
-	      <mass value="1e-5" />
-	      <origin xyz="0 0 0" rpy="0 0 0"/>
-	      <inertia ixx="1e-6" ixy="0" ixz="0" iyy="1e-6" iyz="0" izz="1e-6" />
-	    </inertial>
+    <collision>
+      <origin xyz="0 0 0.025" rpy="0 0 0"/>
+      <geometry>
+        <box size="0.05 0.05 0.05"/>
+      </geometry>
+    </collision>
+    <visual>
+      <origin xyz="0.1 0 0.025" rpy="0 0 0"/>
+      <geometry>
+        <box size="0.25 0.1 0.05"/>
+      </geometry>
+      <material name="red">
+        <color rgba="1 0 0 1"/>
+      </material>
+    </visual>
+    <inertial>
+      <mass value="1e-5" />
+      <origin xyz="0 0 0" rpy="0 0 0"/>
+      <inertia ixx="1e-6" ixy="0" ixz="0" iyy="1e-6" iyz="0" izz="1e-6" />
+    </inertial>
   </link>
   <joint name="camera_joint" type="fixed">
-	    <axis xyz="0 1 0" />
-	    <origin xyz="0.23 0 0.0" rpy="0 0 0"/>
-	    <parent link="link_chassis"/>
-	    <child link="camera_link"/>
-	 </joint>
+    <axis xyz="0 1 0" />
+    <origin xyz="0 0 0.1" rpy="0 0 0"/>
+    <parent link="neck_link"/>
+    <child link="camera_link"/>
+  </joint>
 </robot>

Commit message: make robot visible in rviz

File: urdf/robot.xacro (robot description, xacro)
@@ -163,9 +163,11 @@
     </inertial>
   </link>
-  <joint name="camera_joint" type="fixed">
-    <axis xyz="0 1 0" />
+  <joint name="camera_joint" type="revolute">
+    <axis xyz="0 0 1" />
     <origin xyz="0 0 0.1" rpy="0 0 0"/>
     <parent link="neck_link"/>
     <child link="camera_link"/>
+    <limit effort="10000" velocity="1000" lower="${-pi/4}" upper="${pi/4}"/>
+    <joint_properties damping="1.0" friction="1.0"/>
   </joint>
 </robot>

Commit message: cant get controller running 0> probably namespace issue

File: urdf/robot.xacro (robot description, xacro)
@@ -171,3 +171,13 @@
     <joint_properties damping="1.0" friction="1.0"/>
   </joint>
+  <transmission name="camera_joint_trans">
+    <type>transmission_interface/SimpleTransmission</type>
+    <joint name="camera_joint">
+      <hardwareInterface>EffortJointInterface</hardwareInterface>
+    </joint>
+    <actuator name="motor1">
+      <hardwareInterface>EffortJointInterface</hardwareInterface>
+      <mechanicalInterface>1</mechanicalInterface>
+    </actuator>
+  </transmission>
 </robot>

Commit message: Robot head controllable

File: urdf/robot.xacro (robot description, xacro)
@@ -130,5 +130,5 @@
     </visual>
     <inertial>
-      <mass value="1e-5" />
+      <mass value="0.5" />
       <origin xyz="0 0 0" rpy="0 0 0"/>
       <inertia ixx="1e-6" ixy="0" ixz="0" iyy="1e-6" iyz="0" izz="1e-6" />
@@ -158,5 +158,5 @@
     </visual>
     <inertial>
-      <mass value="1e-5" />
+      <mass value="1" />
       <origin xyz="0 0 0" rpy="0 0 0"/>
       <inertia ixx="1e-6" ixy="0" ixz="0" iyy="1e-6" iyz="0" izz="1e-6" />

Commit message: Implement navigator, not fully working yet

File: urdf/robot.xacro (robot description, xacro)
@@ -9,4 +9,10 @@
       <origin rpy="0 1.5707 1.5707" xyz="0 0 0"/>
       <inertia ixx="0.000526666666667" ixy="0" ixz="0" iyy="0.000526666666667" iyz="0" izz="0.001"/>
+    </inertial>
+  </xacro:macro>
+  <xacro:macro name="cuboid_inertial" params="mass length width height">
+    <inertial>
+      <mass value="${mass}"/>
+      <inertia ixx="${0.83*mass*(width+height)}" ixy="0.0" ixz="0.0" iyy="${0.83*mass*(length+height)}" iyz="0.0" izz="${0.83*mass*(width+length)}" />
     </inertial>
   </xacro:macro>
@@ -157,9 +163,5 @@
       </material>
     </visual>
-    <inertial>
-      <mass value="1" />
-      <origin xyz="0 0 0" rpy="0 0 0"/>
-      <inertia ixx="1e-6" ixy="0" ixz="0" iyy="1e-6" iyz="0" izz="1e-6" />
-    </inertial>
+    <xacro:cuboid_inertial mass="0.3" length="0.25" width="0.1" height="0.05"/>
   </link>
   <joint name="camera_joint" type="revolute">

Commit message: navigator works fine!

File: urdf/robot.xacro (robot description, xacro)
@@ -49,9 +49,5 @@
     <!-- pose and inertial -->
     <pose>0 0 0.1 0 0 0</pose>
-    <inertial>
-      <mass value="5"/>
-      <origin rpy="0 0 0" xyz="0 0 0.1"/>
-      <inertia ixx="0.0395416666667" ixy="0" ixz="0" iyy="0.106208333333" iyz="0" izz="0.106208333333"/>
-    </inertial>
+    <xacro:cuboid_inertial mass="10" length="0.5" width="0.3" height="0.07"/>
     <!-- body -->
     <collision name="collision_chassis">
@@ -66,17 +62,4 @@
       </geometry>
       <material name="blue"/>
-    </visual>
-    <!-- caster front -->
-    <collision name="caster_front_collision">
-      <origin rpy=" 0 0 0" xyz="0.35 0 -0.05"/>
-      <geometry>
-        <sphere radius="0.05"/>
-      </geometry>
-    </collision>
-    <visual name="caster_front_visual">
-      <origin rpy=" 0 0 0" xyz="0.2 0 -0.05"/>
-      <geometry>
-        <sphere radius="0.05"/>
-      </geometry>
     </visual>
   </link>
@@ -106,5 +89,5 @@
   </link>
   <joint name="joint_right_wheel" type="continuous">
-    <origin rpy="0 0 0" xyz="-0.05 0.15 0"/>
+    <origin rpy="0 0 0" xyz="0.2 0.15 -0.03"/>
     <child link="link_right_wheel"/>
     <parent link="link_chassis"/>
@@ -114,5 +97,5 @@
   </joint>
   <joint name="joint_left_wheel" type="continuous">
-    <origin rpy="0 0 0" xyz="-0.05 -0.15 0"/>
+    <origin rpy="0 0 0" xyz="0.2 -0.15 -0.03"/>
     <child link="link_left_wheel"/>
     <parent link="link_chassis"/>
@@ -183,3 +166,52 @@
     </actuator>
   </transmission>
+  <link name="link_castor_axis">
+    <!-- pose and inertial -->
+    <pose>0 0 0.1 0 0 0</pose>
+    <xacro:cuboid_inertial mass="0.2" length="0.05" width="0.035" height="0.03"/>
+    <!-- body -->
+    <collision name="collision_chassis">
+      <origin rpy="0 0 0" xyz="-0.025 0 0"/>
+      <geometry>
+        <box size="0.05 0.035 0.03"/>
+      </geometry>
+    </collision>
+    <visual>
+      <origin rpy="0 0 0" xyz="-0.025 0 0"/>
+      <geometry>
+        <box size="0.05 0.035 0.03"/>
+      </geometry>
+    </visual>
+  </link>
+  <link name="link_castor_wheel">
+    <xacro:default_inertial mass="0.2"/>
+    <collision name="link_castor_wheel_collision">
+      <origin rpy="0 1.5707 1.5707" xyz="0 0 0"/>
+      <geometry>
+        <cylinder length="0.02" radius="0.03"/>
+      </geometry>
+    </collision>
+    <visual name="link_right_wheel_visual">
+      <origin rpy="0 1.5707 1.5707" xyz="0 0 0"/>
+      <geometry>
+        <cylinder length="0.02" radius="0.03"/>
+      </geometry>
+    </visual>
+  </link>
+  <joint name="joint_castor_wheel" type="continuous">
+    <origin rpy="0 0 0" xyz="-0.05 0 -0.015"/>
+    <child link="link_castor_wheel"/>
+    <parent link="link_castor_axis"/>
+    <axis rpy="0 0 0" xyz="0 1 0"/>
+    <limit effort="10000" velocity="1000"/>
+    <joint_properties damping="1.0" friction="1.0"/>
+  </joint>
+  <joint name="joint_castor_axis" type="continuous">
+    <origin rpy="0 0 0" xyz="-0.25 0 -0.05"/>
+    <child link="link_castor_axis"/>
+    <parent link="link_chassis"/>
+    <axis rpy="0 0 0" xyz="0 0 1"/>
+    <limit effort="10000" velocity="1000"/>
+    <joint_properties damping="1.0" friction="1.0"/>
+  </joint>
 </robot>

Commit message: Debug Debug Debug -> Code works completely!

File: urdf/robot.xacro (robot description, xacro)
@@ -192,5 +192,5 @@
       </geometry>
     </collision>
-    <visual name="link_right_wheel_visual">
+    <visual name="link_castor_wheel_visual">
       <origin rpy="0 1.5707 1.5707" xyz="0 0 0"/>
       <geometry>
